Commit message: Added build script for manipulator pkg. Reworked manipulator files. Changed interpreter of grasp_evaluator.py to python2.

File: manipulator/urdf/arm.urdf (robot description, URDF)
Before this commit: robot test_robot, 17 links, 16 joints
Links:
- link base_bracket_right: geometry collision mesh filename=package://manipulator/meshes/base_bracket.stl scale=0.01 0.01 0.01; visual mesh filename=package://manipulator/meshes/base_bracket.stl scale=0.01 0.01 0.01
- link base_link: geometry collision mesh filename=package://manipulator/meshes/base_bracket.stl scale=0.01 0.01 0.01; visual mesh filename=package://manipulator/meshes/base_bracket.stl scale=0.01 0.01 0.01
- link base_servo: geometry collision mesh filename=package://manipulator/meshes/servo.stl scale=0.01 0.01 0.01; visual mesh filename=package://manipulator/meshes/servo.stl scale=0.01 0.01 0.01
- link base_servo_bracket: geometry collision mesh filename=package://manipulator/meshes/servo_bracket.stl scale=0.01 0.01 0.01; visual mesh filename=package://manipulator/meshes/servo_bracket.stl scale=0.01 0.01 0.01
- link base_servo_disc: geometry collision mesh filename=package://manipulator/meshes/servo_disc.stl scale=0.01 0.01 0.01; visual mesh filename=package://manipulator/meshes/servo_disc.stl scale=0.01 0.01 0.01
- link elbow_bracket: geometry collision mesh filename=package://manipulator/meshes/u_bracket.stl scale=0.01 0.01 0.01; visual mesh filename=package://manipulator/meshes/u_bracket.stl scale=0.01 0.01 0.01
- link elbow_servo: geometry collision mesh filename=package://manipulator/meshes/servo.stl scale=0.01 0.01 0.01; visual mesh filename=package://manipulator/meshes/servo.stl scale=0.01 0.01 0.01
- link elbow_servo_bracket: geometry collision mesh filename=package://manipulator/meshes/servo_bracket.stl scale=0.01 0.01 0.01; visual mesh filename=package://manipulator/meshes/servo_bracket.stl scale=0.01 0.01 0.01
- link elbow_servo_disc: geometry collision mesh filename=package://manipulator/meshes/servo_disc.stl scale=0.01 0.01 0.01; visual mesh filename=package://manipulator/meshes/servo_disc.stl scale=0.01 0.01 0.01
- link shoulder2_bracket: geometry collision mesh filename=package://manipulator/meshes/u_bracket.stl scale=0.01 0.01 0.01; visual mesh filename=package://manipulator/meshes/u_bracket.stl scale=0.01 0.01 0.01
- link shoulder2_servo: geometry collision mesh filename=package://manipulator/meshes/servo.stl scale=0.01 0.01 0.01; visual mesh filename=package://manipulator/meshes/servo.stl scale=0.01 0.01 0.01
- link shoulder2_servo_bracket: geometry collision mesh filename=package://manipulator/meshes/servo_bracket.stl scale=0.01 0.01 0.01; visual mesh filename=package://manipulator/meshes/servo_bracket.stl scale=0.01 0.01 0.01
- link shoulder2_servo_disc: geometry collision mesh filename=package://manipulator/meshes/servo_disc.stl scale=0.01 0.01 0.01; visual mesh filename=package://manipulator/meshes/servo_disc.stl scale=0.01 0.01 0.01
- link shoulder_bracket: geometry collision mesh filename=package://manipulator/meshes/u_bracket.stl scale=0.01 0.01 0.01; visual mesh filename=package://manipulator/meshes/u_bracket.stl scale=0.01 0.01 0.01
- link shoulder_servo: geometry collision mesh filename=package://manipulator/meshes/servo.stl scale=0.01 0.01 0.01; visual mesh filename=package://manipulator/meshes/servo.stl scale=0.01 0.01 0.01
- link shoulder_servo_bracket: geometry collision mesh filename=package://manipulator/meshes/servo_bracket.stl scale=0.01 0.01 0.01; visual mesh filename=package://manipulator/meshes/servo_bracket.stl scale=0.01 0.01 0.01
- link shoulder_servo_disc: geometry collision mesh filename=package://manipulator/meshes/servo_disc.stl scale=0.01 0.01 0.01; visual mesh filename=package://manipulator/meshes/servo_disc.stl scale=0.01 0.01 0.01
