Commit message: Move to target position with orientation. Add center point in grasp_detection

File: manipulator/urdf/box_arm.urdf (robot description, URDF)
Before this commit: robot six_dof_arm, 7 links, 6 joints
Joints:
- joint joint1: limit lower=-1.57 upper=1.57 effort=1000.0 velocity=0.5 -> lower=-3.14 upper=3.14 effort=1000.0 velocity=0.5
- joint joint2: limit lower=-1.57 upper=1.57 effort=1000.0 velocity=0.5 -> lower=-3.14 upper=3.14 effort=1000.0 velocity=0.5
- joint joint3: limit lower=-1.57 upper=1.57 effort=1000.0 velocity=0.5 -> lower=-3.14 upper=3.14 effort=1000.0 velocity=0.5
- joint joint4: limit lower=-1.57 upper=1.57 effort=1000.0 velocity=0.5 -> lower=-3.14 upper=3.14 effort=1000.0 velocity=0.5
- joint joint5: limit lower=-1.57 upper=1.57 effort=1000.0 velocity=0.5 -> lower=-3.14 upper=3.14 effort=1000.0 velocity=0.5
- joint joint6: limit lower=-1.57 upper=1.57 effort=1000.0 velocity=0.5 -> lower=-3.14 upper=3.14 effort=1000.0 velocity=0.5

Commit message: Add: new urdf file and setup assistant files

File: manipulator/urdf/box_arm.urdf (robot description, URDF)
Before this commit: robot six_dof_arm, 7 links, 6 joints
Links:
- added link claw_base; collision box size=0.1 0.07 0.05; visual box size=0.1 0.07 0.05
- added link claw_l; collision box size=0.02 0.02 0.1; visual box size=0.02 0.02 0.1
- added link claw_r; collision box size=0.02 0.02 0.1; visual box size=0.02 0.02 0.1
- link link6: geometry visual box size=0.05 0.05 0.05
Joints:
- added joint joint7: type revolute, parent link6, child claw_base, origin xyz=0 0 0.05 rpy=0 0 0, axis 0 1 0, limit lower=-3.14 upper=3.14 effort=1000.0 velocity=0.5
- added joint joint8: type revolute, parent claw_base, child claw_l, origin xyz=0 0 0.05 rpy=0 0 0, axis 0 1 0, limit lower=-3.14 upper=3.14 effort=1000.0 velocity=0.5
- added joint joint9: type revolute, parent claw_base, child claw_r, origin xyz=0 0 0.05 rpy=0 0 0, axis 0 1 0, limit lower=-3.14 upper=3.14 effort=1000.0 velocity=0.5
- joint joint6: origin xyz=0 0 0.1 rpy=0 0 0 -> xyz=0 0 0.075 rpy=0 0 0

Commit message: Fix: changed urdf Add: methods for grasp and release

File: manipulator/urdf/box_arm.urdf (robot description, URDF)
Before this commit: robot six_dof_arm, 10 links, 9 joints
Joints:
- joint joint7: axis 0 1 0 -> (none); limit lower=-3.14 upper=3.14 effort=1000.0 velocity=0.5 -> (none); type revolute -> fixed
